File: PCB_IIm_Ligne.kicad_pcb (KiCad board)
At the start: 2 copper layers, 100 x 100 mm, 18 parts, among them J1 Screw_Terminal_01x08, J2 Screw_Terminal_01x08, J3 Screw_Terminal_01x02, K3 G5V-2_Split, Q1 IRFZ14, U2 NE555DR

Commit message: Schematic V1
Parts:
- removed D1, D8: D, Diode_THT:D_DO-15_P10.16mm_Horizontal
- removed J3: Screw_Terminal_01x02, TerminalBlock_Phoenix:TerminalBlock_Phoenix_MKDS-1,5-2_1x02_P5.00mm_Horizontal
- removed K3: G5V-2_Split, Relay_THT:Relay_DPDT_Omron_G5V-2
- added D3: D, Diode_THT:D_DO-15_P10.16mm_Horizontal, F.Cu at (207.3, 71.4)
- added J4: Screw_Terminal_01x08, TerminalBlock_Phoenix:TerminalBlock_Phoenix_MPT-0,5-8-2.54_1x08_P2.54mm_Horizontal, F.Cu at (50.0, 77.5)
- added J5: Screw_Terminal_01x08, TerminalBlock_Phoenix:TerminalBlock_Phoenix_MKDS-1,5-8-5.08_1x08_P5.08mm_Horizontal, F.Cu at (37.9, 103.5)
- added K1: G2RK-2 DC12, Library:RELAY_G2RK-2_OMR, F.Cu at (165.4, 63.6)
- added K2: Relay_DPDT_Latching_2coil, Package_DIP:DIP-16_W10.16mm_LongPads, F.Cu at (198.6, 71.4)
- added Q2: MPSA56, PCM_Package_TO_SOT_THT_AKL:TO-92_Inline_Wide_EBC, F.Cu at (185.4, 90.2)
- added R1: R, Resistor_THT:R_Axial_DIN0207_L6.3mm_D2.5mm_P10.16mm_Horizontal, F.Cu at (174.0, 72.1)
- added R2: R, Resistor_THT:R_Axial_DIN0207_L6.3mm_D2.5mm_P10.16mm_Horizontal, F.Cu at (174.0, 75.4)
- added R3: R4.7k, Resistor_THT:R_Axial_DIN0207_L6.3mm_D2.5mm_P10.16mm_Horizontal, F.Cu at (178.2, 86.2)
- added R5: R, Resistor_THT:R_Axial_DIN0207_L6.3mm_D2.5mm_P10.16mm_Horizontal, F.Cu at (174.0, 78.7)
- added R6: R, Resistor_THT:R_Axial_DIN0207_L6.3mm_D2.5mm_P10.16mm_Horizontal, F.Cu at (174.0, 82.0)
- J1, J2: footprint TerminalBlock_Phoenix:TerminalBlock_Phoenix_MKDS-1,5-8-5.08_1x08_P5.08mm_Horizontal -> TerminalBlock_Phoenix:TerminalBlock_Phoenix_MPT-0,5-8-2.54_1x08_P2.54mm_Horizontal
- U2: footprint PCM_JLCPCB:SOIC-8_L4.9-W3.9-P1.27-LS6.0-BL -> Package_DIP:DIP-8_W7.62mm_Socket
- moved R8 148.7 mm to (239.4, 13.8), turned to 0 degrees
- moved C2 138.0 mm to (239.8, 11.1)
- moved D6 137.3 mm to (234.9, 8.23), turned to 0 degrees
- moved C1 137.1 mm to (239.8, 8.08), turned to 0 degrees
- moved R7 136.4 mm to (233.5, 14.2)
- moved D7 132.7 mm to (234.9, 11.6), turned to 0 degrees
- moved J1 80.6 mm to (36.8, 113.5), turned to 0 degrees
- moved J2 58.9 mm to (61.5, 82.5), turned to 0 degrees
- moved JP1 55.0 mm to (197.9, 100.8), turned to 0 degrees
- moved D5 34.1 mm to (196.8, 65.0), turned to 90 degrees
- moved D4 34.0 mm to (202.9, 65.0), turned to 90 degrees
- moved D2 30.0 mm to (202.7, 71.4), turned to -90 degrees
- moved Q1 18.2 mm to (174.7, 116.8)
- moved U2 15.3 mm to (160.0, 118.1), turned to 90 degrees
Connections:
- net Traction_P renamed InterrupteurPot2
- D2 pad 1: RelaiBistableSensB -> RelaiBistableSensA
- J1 pad 1: GND -> unconnected-(J1-Pin_1-Pad1)
- J1 pad 2: POT1 -> unconnected-(J1-Pin_2-Pad2)
- J1 pad 3: POT2 -> unconnected-(J1-Pin_3-Pad3)
- J1 pad 4: POT3 -> BoutonSensB
- J1 pad 5: OUT_ARD -> BoutonSensA
- J1 pad 6: Traction_N -> InterrupteurPot1
- J1 pad 8: unconnected-(J1-Pin_8-Pad8) -> VCC
- J2 pad 2: LED_Alim -> GND
- J2 pad 3: LED_SensA -> GND
- J2 pad 4: LED_SensB -> GND
- J2 pad 5: LED_Traction -> LED_Alim
- J2 pad 6: unconnected-(J2-Pin_6-Pad6) -> LED_SensA
- J2 pad 7: unconnected-(J2-Pin_7-Pad7) -> LED_SensB
- J2 pad 8: unconnected-(J2-Pin_8-Pad8) -> LED_TractionEnService
Routing:
- net POT3: track 46.0 -> 0.00 mm
- net GATE: track 10.6 -> 0.00 mm
- net Net-(U2-DISCH): track 10.6 -> 0.00 mm
- net OUT: track 9.95 -> 0.00 mm
- net Net-(U2-CONT): track 4.17 -> 0.00 mm
- net GND: track 3.42 -> 0.00 mm
- net VCC: track 2.31 -> 0.00 mm
- added copper zone on B.Cu, net GND

Commit message: Schematic V2 + BOM
Parts:
- removed D5: D, Diode_THT:D_DO-15_P10.16mm_Horizontal
- removed D6, D7: 1N4001W, PCM_JLCPCB:D_SOD-123FL
- removed J5: Screw_Terminal_01x08, TerminalBlock_Phoenix:TerminalBlock_Phoenix_MKDS-1,5-8-5.08_1x08_P5.08mm_Horizontal
- removed U2: NE555DR, Package_DIP:DIP-8_W7.62mm_Socket
- added C5: C100nF, Capacitor_THT:C_Rect_L7.5mm_W6.5mm_P5.00mm, F.Cu at (114.5, 58.7)
- added C6: C100nF, Capacitor_THT:C_Rect_L7.5mm_W6.5mm_P5.00mm, F.Cu at (114.5, 66.8)
- added D1: D, Diode_THT:D_DO-15_P10.16mm_Horizontal, F.Cu at (62.5, 55.4)
- added J3: Screw_Terminal_01x08, TerminalBlock_Phoenix:TerminalBlock_Phoenix_MKDS-1,5-8-5.08_1x08_P5.08mm_Horizontal, F.Cu at (39.9, 119.4)
- added OC1: 6N137, PCM_Package_DIP_AKL:DIP-8_W7.62mm_Socket_LongPads, F.Cu at (101.2, 45.0)
- added OC2: 6N137, PCM_Package_DIP_AKL:DIP-8_W7.62mm_Socket_LongPads, F.Cu at (113.0, 45.0)
- added OC3: 6N137, PCM_Package_DIP_AKL:DIP-8_W7.62mm_Socket_LongPads, F.Cu at (124.7, 45.0)
- added Q3: IRF9540N, PCM_Package_TO_SOT_THT_AKL:TO-220-3_Vertical_GDS, F.Cu at (124.7, 58.6)
- added Q4: IRF9540N, PCM_Package_TO_SOT_THT_AKL:TO-220-3_Vertical_GDS, F.Cu at (124.7, 64.6)
- added R10: R100, Resistor_THT:R_Axial_DIN0207_L6.3mm_D2.5mm_P10.16mm_Horizontal, F.Cu at (100.7, 56.7)
- added R11: R100, Resistor_THT:R_Axial_DIN0207_L6.3mm_D2.5mm_P10.16mm_Horizontal, F.Cu at (100.7, 60.8)
- added R12: R4.7k, Resistor_THT:R_Axial_DIN0207_L6.3mm_D2.5mm_P10.16mm_Horizontal, F.Cu at (100.7, 64.8)
- added R13: R4.7k, Resistor_THT:R_Axial_DIN0207_L6.3mm_D2.5mm_P10.16mm_Horizontal, F.Cu at (100.7, 68.9)
- added R14: R, Resistor_THT:R_Axial_DIN0207_L6.3mm_D2.5mm_P10.16mm_Horizontal, F.Cu at (100.7, 72.9)
- added R15: R, Resistor_THT:R_Axial_DIN0207_L6.3mm_D2.5mm_P10.16mm_Horizontal, F.Cu at (100.7, 77.0)
- added R16: R, Resistor_THT:R_Axial_DIN0207_L6.3mm_D2.5mm_P10.16mm_Horizontal, F.Cu at (100.7, 81.0)
- added R4: R4.7k, Resistor_THT:R_Axial_DIN0207_L6.3mm_D2.5mm_P10.16mm_Horizontal, F.Cu at (89.7, 115.6)
- added R9: R100, Resistor_THT:R_Axial_DIN0207_L6.3mm_D2.5mm_P10.16mm_Horizontal, F.Cu at (58.7, 92.7)
- added U1: NE555DR, Package_DIP:DIP-8_W7.62mm_Socket, F.Cu at (64.8, 120.9)
- C1: value 100nF -> C100nF; footprint PCM_JLCPCB:C_0805 -> Capacitor_THT:C_Rect_L7.5mm_W6.5mm_P5.00mm
- C2: value 1nF -> C1nF; footprint PCM_JLCPCB:C_0805 -> Capacitor_THT:C_Rect_L7.5mm_W6.5mm_P5.00mm
- Q1: value IRFZ14 -> STP80NF12
- R7: value 1kΩ -> R1k; footprint PCM_JLCPCB:R_0402 -> Resistor_THT:R_Axial_DIN0207_L6.3mm_D2.5mm_P10.16mm_Horizontal
- R8: value 5.1kΩ -> R4.7k; footprint PCM_JLCPCB:R_0603 -> Resistor_THT:R_Axial_DIN0207_L6.3mm_D2.5mm_P10.16mm_Horizontal
- moved R8 212.2 mm to (55.1, 118.9), turned to 180 degrees
- moved C2 198.3 mm to (80.0, 128.5)
- moved C1 195.6 mm to (80.0, 121.0)
- moved R7 185.9 mm to (76.2, 113.3), turned to -90 degrees
- moved D3 171.0 mm to (45.2, 126.0), turned to 0 degrees
- moved D4 161.3 mm to (55.4, 130.1), turned to 180 degrees
- moved Q2 146.4 mm to (49.5, 144.5)
- moved D2 140.7 mm to (62.5, 59.9), turned to 0 degrees
- moved JP1 139.2 mm to (58.6, 98.8)
- moved R3 138.1 mm to (45.0, 122.2)
- moved K2 136.3 mm to (62.5, 64.0), turned to 0 degrees
- moved Q1 126.9 mm to (51.1, 88.1), turned to 0 degrees
- moved R1 123.5 mm to (55.1, 105.7)
- moved R2 123.5 mm to (55.1, 109.0)
- moved R5 123.5 mm to (55.1, 112.3)
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Connections:
- D3 pad 1: RelaiBistableSensB -> POT1
- D3 pad 2: GND -> Net-(D3-A)
- D4 pad 1: RelaiBistableSensB -> Net-(D3-A)
- D4 pad 2: GND -> POT2
- J1 pad 2: unconnected-(J1-Pin_2-Pad2) -> RelaiBistableSensA
- J1 pad 3: unconnected-(J1-Pin_3-Pad3) -> RelaiBistableSensB
- J1 pad 4: BoutonSensB -> RelaiBistableSensA
- J1 pad 5: BoutonSensA -> RelaiBistableSensB
- JP1 pad 3: OUT_ARD -> CommandeTractionArduino
- Q1 pad 1: GATE -> Net-(Q1-G)
- R7 pad 2: Net-(U2-DISCH) -> Net-(D3-A)
Routing:
- net SensB: track 0.00 -> 50.9 mm, vias 0 -> 1
- net Traction_P: track 0.00 -> 47.2 mm
- net SensA: track 0.00 -> 42.5 mm, vias 0 -> 1
- net RAIL_2: track 0.00 -> 40.4 mm
- net RAIL_1: track 0.00 -> 37.4 mm
- net Traction_N: track 0.00 -> 27.6 mm
- net LED_TractionEnService: track 0.00 -> 25.8 mm
- net LED_SensB: track 0.00 -> 25.1 mm
- net LED_SensA: track 0.00 -> 24.3 mm
- net LED_Alim: track 0.00 -> 23.6 mm
- net RelaiBistableSensB: track 0.00 -> 15.7 mm
- net Interrupteur2: track 0.00 -> 12.9 mm
- net RelaiBistableSensA: track 0.00 -> 10.8 mm
- net GATE: track 0.00 -> 6.11 mm
- net Net-(Q1-G): track 0.00 -> 5.62 mm
- added copper zone on F.Cu, net VCC

Commit message: Schematic V1
Parts:
- removed C1: C100nF, Capacitor_THT:C_Rect_L7.5mm_W6.5mm_P5.00mm
- removed C2: C1nF, Capacitor_THT:C_Rect_L7.5mm_W6.5mm_P5.00mm
- removed OC2, OC3: 6N137, PCM_Package_DIP_AKL:DIP-8_W7.62mm_Socket_LongPads
- removed Q1: STP80NF12, PCM_Package_TO_SOT_THT_AKL:TO-220-3_Vertical_GDS
- removed R16: R, Resistor_THT:R_Axial_DIN0207_L6.3mm_D2.5mm_P10.16mm_Horizontal
- removed R9: R100, Resistor_THT:R_Axial_DIN0207_L6.3mm_D2.5mm_P10.16mm_Horizontal
- removed U1: NE555DR, Package_DIP:DIP-8_W7.62mm_Socket
- added C7: C100nF, Capacitor_THT:C_Rect_L7.5mm_W6.5mm_P5.00mm, F.Cu at (88.1, 52.2)
- added DZ1: 1N4733A, PCM_Diode_THT_AKL:D_DO-41_SOD81_P10.16mm_Horizontal_Zener, F.Cu at (79.6, 93.7)
- added JP2: SolderJumper_2_Bridged, Jumper:SolderJumper-2_P1.3mm_Bridged_RoundedPad1.0x1.5mm, F.Cu at (160.3, 46.2)
- added Q5: 2N3904, PCM_Package_TO_SOT_THT_AKL:TO-92_Inline_Wide_EBC, F.Cu at (170.3, 38.9)
- added Q6: IRF40B207, PCM_Package_TO_SOT_THT_AKL:TO-220-3_Vertical_GDS, F.Cu at (184.3, 49.7)
- added U2: TLC555xP, PCM_Package_DIP_AKL:DIP-8_W7.62mm_LongPads, F.Cu at (105.4, 92.4)
- C6: value C100nF -> C1nF
- OC1: footprint PCM_Package_DIP_AKL:DIP-8_W7.62mm_Socket_LongPads -> PCM_Package_DIP_AKL:DIP-8_W7.62mm_LongPads
- Q3, Q4: value IRF9540N -> BC557B; footprint PCM_Package_TO_SOT_THT_AKL:TO-220-3_Vertical_GDS -> PCM_Package_TO_SOT_THT_AKL:TO-92_Inline_Wide_CBE
- R10, R11: value R100 -> R
- R12, R8: value R4.7k -> R1k
- R13: value R4.7k -> R10k
- R14: value R -> R10k
- R15: value R -> R100
- moved Q2 119.0 mm to (96.6, 35.3), turned to 0 degrees
- moved R4 82.6 mm to (42.9, 47.5), turned to 0 degrees
- moved R3 78.8 mm to (42.9, 43.5)
- moved R15 72.2 mm to (167.6, 49.7)
- moved R1 71.4 mm to (42.9, 35.4), turned to 0 degrees
- moved R2 70.6 mm to (42.9, 39.4), turned to 0 degrees
- moved R13 70.5 mm to (167.6, 46.6)
- moved R12 70.2 mm to (167.6, 43.5)
- moved R14 69.8 mm to (167.5, 52.8)
- moved D3 65.1 mm to (93.8, 82.6)
- moved R7 63.1 mm to (42.9, 59.6), turned to 0 degrees
- moved R5 61.9 mm to (42.9, 51.5), turned to 0 degrees
- moved J3 61.7 mm to (66.8, 63.8), turned to 0 degrees
- moved R6 61.2 mm to (42.9, 55.6), turned to 0 degrees
- moved R10 59.7 mm to (42.9, 71.8)
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Connections:
- C5 pad 1: VCC -> POT3
- C6 pad 1: VCC -> Net-(U2-CV)
- J3 pad 1: GND -> RAIL_2
- J3 pad 2: GND -> RAIL_1
- J3 pad 3: Traction_P -> VCC
- J3 pad 4: Traction_P -> VCC
- J3 pad 5: VCC -> Traction_P
- J3 pad 6: VCC -> Traction_P
- J3 pad 7: RAIL_1 -> GND
- J3 pad 8: RAIL_2 -> GND
- OC1 pad 2: Net-(R14--) -> unconnected-(OC1-Pad2)
- OC1 pad 3: GND -> unconnected-(OC1-Pad3)
- OC1 pad 6: Net-(R10-+) -> Net-(R12-+)
- OC1 pad 7: VCC -> Net-(JP2-A)
- OC1 pad 8: VCC -> +5V
- Q3 pad 1: Net-(Q3-G) -> RelaiBistableSensA
- Q3 pad 2: RelaiBistableSensA -> Net-(Q3-B)
- Q4 pad 1: Net-(Q4-G) -> RelaiBistableSensB
- Q4 pad 2: RelaiBistableSensB -> Net-(Q4-B)
- R10 pad 1: Net-(R10-+) -> CommandeRelaiArdA
- R10 pad 2: Net-(Q3-G) -> Net-(Q3-B)
- R11 pad 1: Net-(R11-+) -> CommandeRelaiArdB
- R11 pad 2: Net-(Q4-G) -> Net-(Q4-B)
- R12 pad 1: Net-(Q3-G) -> Net-(R12-+)
- R12 pad 2: VCC -> Net-(Q5-B)
- R13 pad 1: Net-(Q4-G) -> GND
- R13 pad 2: VCC -> Net-(Q5-B)
- R14 pad 1: CommandeSensA -> Net-(Q5-E)
- R14 pad 2: Net-(R14--) -> VCC
- R15 pad 1: CommandeSensB -> Net-(Q5-E)
- R8 pad 1: OUT -> VCC
- R8 pad 2: GND -> +5V
Routing:
- net SensB: track 50.9 -> 0.00 mm, vias 1 -> 0
- net Traction_P: track 47.2 -> 0.00 mm
- net SensA: track 42.5 -> 0.00 mm, vias 1 -> 0
- net RAIL_2: track 40.4 -> 0.00 mm
- net RAIL_1: track 37.4 -> 0.00 mm
- net Traction_N: track 27.6 -> 0.00 mm
- net LED_TractionEnService: track 25.8 -> 0.00 mm
- net LED_SensB: track 25.1 -> 0.00 mm
- net LED_SensA: track 24.3 -> 0.00 mm
- net LED_Alim: track 23.6 -> 0.00 mm
- net RelaiBistableSensB: track 15.7 -> 0.00 mm
- net Interrupteur2: track 12.9 -> 0.00 mm
- net RelaiBistableSensA: track 10.8 -> 0.00 mm
- net GATE: track 6.11 -> 0.00 mm
- net Net-(Q1-G): track 5.62 -> 0.00 mm
- removed copper zone on B.Cu, net GND
- removed copper zone on F.Cu, net VCC

Commit message: Schematic V2
Parts:
- removed DZ1: 1N4733A, PCM_Diode_THT_AKL:D_DO-41_SOD81_P10.16mm_Horizontal_Zener
- removed JP2: SolderJumper_2_Bridged, Jumper:SolderJumper-2_P1.3mm_Bridged_RoundedPad1.0x1.5mm
- removed OC1: 6N137, PCM_Package_DIP_AKL:DIP-8_W7.62mm_LongPads
- removed R8: R1k, Resistor_THT:R_Axial_DIN0207_L6.3mm_D2.5mm_P10.16mm_Horizontal
- added H1: MountingHole, MountingHole:MountingHole_3.2mm_M3, F.Cu at (200.9, 86.7)
- added H2: MountingHole, MountingHole:MountingHole_3.2mm_M3, F.Cu at (228.3, 90.0)
- added H3: MountingHole, MountingHole:MountingHole_3.2mm_M3, F.Cu at (228.3, 98.0)
- added H4: MountingHole, MountingHole:MountingHole_3.2mm_M3, F.Cu at (228.3, 105.9)
- moved R4 128.4 mm to (169.3, 70.4), turned to 90 degrees
- moved R3 124.4 mm to (166.2, 60.2), turned to -90 degrees
- moved JP1 124.1 mm to (2.33, 1.27)
- moved R10 120.8 mm to (163.1, 60.2), turned to -90 degrees
- moved R11 118.2 mm to (160.1, 60.2), turned to -90 degrees
- moved R7 110.7 mm to (153.5, 53.8), turned to 90 degrees
- moved R6 96.7 mm to (139.4, 60.9), turned to -90 degrees
- moved R5 93.9 mm to (136.4, 60.9), turned to -90 degrees
- moved R2 93.0 mm to (133.4, 60.9), turned to -90 degrees
- moved R1 91.1 mm to (130.4, 60.9), turned to -90 degrees
- moved Q2 86.1 mm to (169.8, 80.6), turned to 90 degrees
- moved K2 82.8 mm to (158.5, 97.0)
- moved Q3 79.0 mm to (165.0, 80.6), turned to 90 degrees
- moved K1 78.3 mm to (150.7, 114.1)
- moved D4 75.7 mm to (161.5, 53.9), turned to 90 degrees
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Connections:
- J3 pad 1: RAIL_2 -> VCC
- J3 pad 2: RAIL_1 -> VCC
- J3 pad 3: VCC -> +20V
- J3 pad 4: VCC -> +20V
- J3 pad 5: Traction_P -> RAIL_2
- J3 pad 6: Traction_P -> RAIL_1
- K1 pad 3: Traction_N -> GND
- K1 pad 6: Traction_N -> GND
- Q6 pad 2: VCC -> +20V
- R12 pad 1: Net-(R12-+) -> CommandetTraction
- U2 pad 3: unconnected-(U2-Q-Pad3) -> CommandetTraction
Routing:
- net RelaiBistableSensB: track 0.00 -> 93.6 mm
- net RelaiBistableSensA: track 0.00 -> 87.7 mm
- net AlimBoutonSens: track 0.00 -> 60.7 mm
- net Traction_P: track 0.00 -> 43.1 mm
- net +20V: track 0.00 -> 35.5 mm
- net Interrupteur2: track 0.00 -> 31.2 mm
- net RAIL_1: track 0.00 -> 26.3 mm
- net Net-(D3-A): track 0.00 -> 21.5 mm
- net RAIL_2: track 0.00 -> 18.9 mm
- net LED_TractionEnService: track 0.00 -> 17.6 mm
- net Net-(Q5-B): track 0.00 -> 14.1 mm, vias 0 -> 1
- net LED_SensB: track 0.00 -> 13.5 mm
- net Net-(Q5-E): track 0.00 -> 10.8 mm
- net Net-(Q6-G): track 0.00 -> 10.0 mm
- net CommandetTraction: track 0.00 -> 9.93 mm
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- added copper zone on B.Cu, net GND
- added copper zone on F.Cu, net VCC
