File: PCB_IIm_Ligne.kicad_pcb (KiCad board)
At the start: 2 copper layers, 80 x 80 mm, 32 parts, among them J1 Screw_Terminal_01x08, J2 Screw_Terminal_01x08, J3 Screw_Terminal_01x08, K1 G2RK-2 DC12, K2 Relay_DPDT_Latching_2coil

Commit message: recomit
Routing:
- net Net-(D3-A): track 16.4 -> 12.3 mm
- net RAIL_2: track 18.0 -> 17.0 mm
Changed lines of the file:
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@@
+	)
+	(segment
+		(start 173.736 80.01)
+		(end 173.736001 83.058)
+		(width 0.2)
+		(layer "F.Cu")
+		(net "Interrupteur")
+	)
+	(segment
+		(start 173.736001 83.058)
+		(end 173.736001 86.105998)
+		(width 0.2)
+		(layer "F.Cu")
+		(net "Interrupteur")
+	)
+	(segment
+		(start 173.736001 86.105998)
+		(end 173.735999 86.106)
+		(width 0.2)
+		(layer "F.Cu")
+		(net "Interrupteur")
+	)
+	(segment
+		(start 171.38 57.404)
+		(end 176.53 52.254)
+		(width 0.2)
+		(layer "F.Cu")
+		(net "Net-(D3-A)")
+	)
+	(segment
+		(start 166.37 57.404)
+		(end 171.38 57.404)
+		(width 0.2)
+		(layer "F.Cu")
+		(net "Net-(D3-A)")
+	)
+	(segment
+		(start 194.564 60.706)
+		(end 192.024 58.166)
+		(width 0.2)
+		(layer "F.Cu")
+		(net "RelaiBistableSensA")
+	)
+	(segment
+		(start 192.024 47.665995)
+		(end 189.630005 45.272)
+		(width 0.2)
+		(layer "F.Cu")
+		(net "RelaiBistableSensA")
+	)
+	(segment
+		(start 194.564 69.088)
+		(end 194.564 60.706)
+		(width 0.2)
+		(layer "F.Cu")
+		(net "RelaiBistableSensA")
+	)
+	(segment
+		(start 187.658005 47.244)
+		(end 189.630005 45.272)
+		(width 0.2)
+		(layer "F.Cu")
+		(net "RelaiBistableSensA")
+	)
+	(segment
+		(start 192.278 73.659999)
+		(end 192.278 71.374)
+		(width 0.2)
+		(layer "F.Cu")
+		(net "RelaiBistableSensA")
+	)
+	(segment
+		(start 192.024 58.166)
+		(end 192.024 47.665995)
+		(width 0.2)
+		(layer "F.Cu")
+		(net "RelaiBistableSensA")
+	)
+	(segment
+		(start 158.242 47.244)
+		(end 187.658005 47.244)
+		(width 0.2)
+		(layer "F.Cu")
+		(net "RelaiBistableSensA")
+	)
+	(segment
+		(start 192.278 73.659999)
+		(end 197.108999 73.659999)
+		(width 0.2)
+		(layer "F.Cu")
+		(net "RelaiBistableSensA")
+	)
+	(segment
+		(start 189.062004 44.703999)
+		(end 189.630005 45.272)
+		(width 0.2)
+		(layer "F.Cu")
+		(net "RelaiBistableSensA")
+	)
+	(segment
+		(start 192.278 71.374)
+		(end 194.564 69.088)
+		(width 0.2)
+		(layer "F.Cu")
+		(net "RelaiBistableSensA")
+	)
+	(segment
+		(start 197.108999 73.659999)
+		(end 197.358 73.909)
+		(width 0.2)
+		(layer "F.Cu")
+		(net "RelaiBistableSensA")
 	)
 	(segment
@@
 	)
 	(segment
-		(start 194.564 60.706)
-		(end 192.024 58.166)
-		(width 0.2)
-		(layer "F.Cu")
-		(net "RelaiBistableSensA")
-	)
-	(segment
-		(start 192.024 47.665995)
-		(end 189.630005 45.272)
-		(width 0.2)
-		(layer "F.Cu")
-		(net "RelaiBistableSensA")
-	)
-	(segment
-		(start 194.564 69.088)
-		(end 194.564 60.706)
-		(width 0.2)
-		(layer "F.Cu")
-		(net "RelaiBistableSensA")
-	)
-	(segment
-		(start 187.658005 47.244)
-		(end 189.630005 45.272)
-		(width 0.2)
-		(layer "F.Cu")
-		(net "RelaiBistableSensA")
-	)
-	(segment
-		(start 192.278 73.659999)
-		(end 192.278 71.374)
-		(width 0.2)
-		(layer "F.Cu")
-		(net "RelaiBistableSensA")
-	)
-	(segment
-		(start 192.024 58.166)
-		(end 192.024 47.665995)
-		(width 0.2)
-		(layer "F.Cu")
-		(net "RelaiBistableSensA")
-	)
-	(segment
-		(start 158.242 47.244)
-		(end 187.658005 47.244)
-		(width 0.2)
-		(layer "F.Cu")
-		(net "RelaiBistableSensA")
-	)
-	(segment
-		(start 192.278 73.659999)
-		(end 197.108999 73.659999)
-		(width 0.2)
-		(layer "F.Cu")
-		(net "RelaiBistableSensA")
-	)
-	(segment
-		(start 189.062004 44.703999)
-		(end 189.630005 45.272)
-		(width 0.2)
-		(layer "F.Cu")
-		(net "RelaiBistableSensA")
-	)
-	(segment
-		(start 192.278 71.374)
-		(end 194.564 69.088)
-		(width 0.2)
-		(layer "F.Cu")
-		(net "RelaiBistableSensA")
-	)
-	(segment
-		(start 197.108999 73.659999)
-		(end 197.358 73.909)
-		(width 0.2)
-		(layer "F.Cu")
-		(net "RelaiBistableSensA")
+		(start 173.99 77.216)
+		(end 201.671 77.216)
+		(width 0.2)
+		(layer "F.Cu")
+		(net "SensA")
+	)
+	(segment
+		(start 173.736 76.962)
+		(end 173.99 77.216)
+		(width 0.2)
+		(layer "F.Cu")
+		(net "SensA")
+	)
+	(segment
+		(start 201.671 77.216)
+		(end 204.978 73.909)
+		(width 0.2)
+		(layer "F.Cu")
+		(net "SensA")
+	)
+	(segment
+		(start 199.644 76.708)
+		(end 201.168 75.184)
+		(width 0.2)
+		(layer "F.Cu")
+		(net "SensB")
+	)
+	(segment
+		(start 204.978 68.58)
+		(end 204.978 63.749)
+		(width 0.2)
+		(layer "F.Cu")
+		(net "SensB")
+	)
+	(segment
+		(start 176.53 76.708)
+		(end 199.644 76.708)
+		(width 0.2)
+		(layer "F.Cu")
+		(net "SensB")
+	)
+	(segment
+		(start 201.168 75.184)
+		(end 201.168 72.39)
+		(width 0.2)
+		(layer "F.Cu")
+		(net "SensB")
+	)
+	(segment
+		(start 201.168 72.39)
+		(end 204.978 68.58)
+		(width 0.2)
+		(layer "F.Cu")
+		(net "SensB")
+	)
+	(segment
+		(start 173.736 73.914)
+		(end 176.53 76.708)
+		(width 0.2)
+		(layer "F.Cu")
+		(net "SensB")
 	)
 	(segment
@@
 	)
 	(segment
-		(start 171.38 57.404)
-		(end 176.53 52.254)
-		(width 0.2)
-		(layer "F.Cu")
-		(net "Net-(D3-A)")
-	)
-	(segment
-		(start 166.37 57.404)
-		(end 171.38 57.404)
-		(width 0.2)
-		(layer "F.Cu")
-		(net "Net-(D3-A)")
-	)
-	(segment
-		(start 192.023999 33.02)
-		(end 192.024 28.956)
-		(width 0.2)
-		(layer "F.Cu")
-		(net "Net-(D3-A)")
+		(start 213.126004 49.276)
+		(end 221.996 49.276)
+		(width 2)
+		(layer "F.Cu")
+		(net "RAIL_2")
 	)
 	(segment
@@
 	)
 	(segment
-		(start 211.582 49.276)
-		(end 221.996 49.276)
+		(start 209.630005 52.771999)
+		(end 213.126004 49.276)
 		(width 2)
 		(layer "F.Cu")
@@
 	)
 	(segment
-		(start 209.630005 52.771999)
-		(end 209.630005 51.227995)
-		(width 2)
-		(layer "F.Cu")
-		(net "RAIL_2")
-	)
-	(segment
-		(start 209.630005 51.227995)
-		(end 211.582 49.276)
-		(width 2)
-		(layer "F.Cu")
-		(net "RAIL_2")
+		(start 207.999003 48.641)
+		(end 210.499006 48.641)
+		(width 2)
+		(layer "B.Cu")
+		(net "Traction_P")
+	)
+	(segment
+		(start 204.630003 45.272)
+		(end 207.999003 48.641)
+		(width 2)
+		(layer "B.Cu")
+		(net "Traction_P")
+	)
+	(segment
+		(start 210.499006 48.641)
+		(end 214.630006 52.772)
+		(width 2)
+		(layer "B.Cu")
+		(net "Traction_P")
 	)
 	(segment
@@
 	)
 	(segment
-		(start 173.99 77.216)
-		(end 201.671 77.216)
-		(width 0.2)
-		(layer "F.Cu")
-		(net "SensA")
-	)
-	(segment
-		(start 173.736 76.962)
-		(end 173.99 77.216)
-		(width 0.2)
-		(layer "F.Cu")
-		(net "SensA")
-	)
-	(segment
-		(start 201.671 77.216)
-		(end 204.978 73.909)
-		(width 0.2)
-		(layer "F.Cu")
-		(net "SensA")
-	)
-	(segment
 		(start 163.322 76.708)
 		(end 163.576 76.962)
@@
 		(net "LED_TractionEnService")
 	)
-	(segment
-		(start 199.644 76.708)
-		(end 201.168 75.184)
-		(width 0.2)
-		(layer "F.Cu")
-		(net "SensB")
-	)
-	(segment
-		(start 204.978 68.58)
-		(end 204.978 63.749)
-		(width 0.2)
-		(layer "F.Cu")
-		(net "SensB")
-	)
-	(segment
-		(start 176.53 76.708)
-		(end 199.644 76.708)
-		(width 0.2)
-		(layer "F.Cu")
-		(net "SensB")
-	)
-	(segment
-		(start 201.168 75.184)
-		(end 201.168 72.39)
-		(width 0.2)
-		(layer "F.Cu")
-		(net "SensB")
-	)
-	(segment
-		(start 201.168 72.39)
-		(end 204.978 68.58)
-		(width 0.2)
-		(layer "F.Cu")
-		(net "SensB")
-	)
-	(segment
-		(start 173.736 73.914)
-		(end 176.53 76.708)
-		(width 0.2)
-		(layer "F.Cu")
-		(net "SensB")
-	)
-	(segment
-		(start 211.134006 49.276)
-		(end 214.630006 52.772)
-		(width 2)
-		(layer "B.Cu")
-		(net "Traction_P")
-	)
-	(segment
-		(start 208.634003 49.276)
-		(end 211.134006 49.276)
-		(width 2)
-		(layer "B.Cu")
-		(net "Traction_P")
-	)
-	(segment
-		(start 204.630003 45.272)
-		(end 208.634003 49.276)
-		(width 2)
-		(layer "B.Cu")
-		(net "Traction_P")
-	)
-	(segment
-		(start 173.736 80.01)
-		(end 173.736001 83.058)
-		(width 0.2)
-		(layer "F.Cu")
-		(net "Interrupteur")
-	)
-	(segment
-		(start 173.736001 83.058)
-		(end 173.736001 86.105998)
-		(width 0.2)
-		(layer "F.Cu")
-		(net "Interrupteur")
-	)
-	(segment
-		(start 173.736001 86.105998)
-		(end 173.735999 86.106)
-		(width 0.2)
-		(layer "F.Cu")
-		(net "Interrupteur")
-	)
 	(embedded_fonts no)

Commit message: Finder relay Lib
Parts:
- removed K1: G2RK-2 DC12, Library:RELAY_G2RK-2_OMR
- added D5: D, Diode_THT:D_DO-15_P10.16mm_Horizontal, F.Cu at (251.2, 67.2)
- added J4: Screw_Terminal_01x08, TerminalBlock_Phoenix:TerminalBlock_Phoenix_MPT-0,5-8-2.54_1x08_P2.54mm_Horizontal, F.Cu at (251.8, 60.2)
- added K3: ~, Library_IIm:Finder_41.52.6.012.4016, F.Cu at (203.5, 49.6)
- R13, R14: value R10k -> 10K
- R18, R9: value 260 -> 270
- R4: value 220 -> 1K
- R7: value R1k -> 470
- renumbered C7 to C3, C6 to C4

Commit message: Modif Schematic + Layout
Parts:
- removed K3: ~, Library_IIm:Finder_41.52.6.012.4016
- added K1: ~, Library_IIm:Finder_41.52.6.012.4016, F.Cu at (203.9, 54.3)
- moved D5 42.6 mm to (215.1, 44.6), turned to 180 degrees
Connections:
- D1 pad 1: RelaiBistableSensB -> VCC
- D1 pad 2: GND -> RelaiBistableSensA_N
- D2 pad 1: RelaiBistableSensA -> VCC
- D2 pad 2: GND -> RelaiBistableSensB_N
- J3 pad 5: +20V -> RAIL_2
- J3 pad 6: +20V -> RAIL_1
- J3 pad 7: RAIL_2 -> +20V
- J3 pad 8: RAIL_1 -> +20V
- K2 pad 1: RelaiBistableSensA -> VCC
- K2 pad 2: RelaiBistableSensB -> VCC
Routing:
- net RelaiBistableSensB: track 84.3 -> 0.00 mm
- net RelaiBistableSensA: track 69.6 -> 0.00 mm
- net Traction_P: track 13.1 -> 0.00 mm
- net RelaiBistableSensA_N: track 0.00 -> 11.9 mm
- net RelaiBistableSensB_N: track 0.00 -> 9.74 mm
- net RAIL_2: track 17.0 -> 16.2 mm
- added copper zone on F.Cu, net +20V
- added copper zone on B.Cu, net GND
- added copper zone on F.Cu, net Traction_P
- added copper zone on F.Cu, net VCC

Commit message: kicad modif
Parts:
- added D6: D_Zener, Diode_THT:D_DO-15_P10.16mm_Horizontal, F.Cu at (215.1, 40.2)
- added R3: 1R 2W, Resistor_THT:R_Axial_DIN0411_L9.9mm_D3.6mm_P12.70mm_Horizontal, F.Cu at (215.1, 36.0)
- moved R9 140.2 mm to (163.6, 67.8)
- moved R10 139.4 mm to (163.6, 64.8)
- moved D4 18.8 mm to (174.4, 40.4)
- moved R7 18.8 mm to (184.6, 44.5)
- moved D3 18.8 mm to (174.4, 35.3)
Connections:
- J4 pad 1: unconnected-(J4-Pin_1-Pad1) -> ResistanceShunt
Routing:
- net RAIL_2: track 16.2 -> 0.00 mm
- net RAIL_1: track 15.7 -> 0.00 mm
- net RelaiBistableSensB_N: track 9.74 -> 24.5 mm
- net Net-(D3-A): track 12.3 -> 0.00 mm
- net RelaiBistableSensA_N: track 11.9 -> 19.1 mm

Commit message: Kicad Modification
Parts:
- removed C3: 100nF, Capacitor_THT:C_Rect_L7.5mm_W6.5mm_P5.00mm
- removed C4: C1nF, Capacitor_THT:C_Rect_L7.5mm_W6.5mm_P5.00mm
- removed C5: 270nF, Capacitor_THT:C_Rect_L7.5mm_W6.5mm_P5.00mm
- removed D1, D2, D3, D4, D5: D, Diode_THT:D_DO-15_P10.16mm_Horizontal
- removed D6: D_Zener, Diode_THT:D_DO-15_P10.16mm_Horizontal
- removed H1, H2, H3, H4: MountingHole, MountingHole:MountingHole_3.2mm_M3
- removed J1, J2, J4: Screw_Terminal_01x08, TerminalBlock_Phoenix:TerminalBlock_Phoenix_MPT-0,5-8-2.54_1x08_P2.54mm_Horizontal
- removed J3: Screw_Terminal_01x08, TerminalBlock_Phoenix:TerminalBlock_Phoenix_MKDS-1,5-8-5.08_1x08_P5.08mm_Horizontal
- removed K1: ~, Library_IIm:Finder_41.52.6.012.4016
- removed K2: Relay_DPDT_Latching_2coil, Package_DIP:DIP-16_W10.16mm_LongPads
- removed R1, R2, R5, R6: R, Resistor_THT:R_Axial_DIN0207_L6.3mm_D2.5mm_P10.16mm_Horizontal
- removed R10, R19, R8: 10k, Resistor_THT:R_Axial_DIN0207_L6.3mm_D2.5mm_P10.16mm_Horizontal
- removed R12, R15, R4: 1K, Resistor_THT:R_Axial_DIN0207_L6.3mm_D2.5mm_P10.16mm_Horizontal
- removed R13, R14: 10K, Resistor_THT:R_Axial_DIN0207_L6.3mm_D2.5mm_P10.16mm_Horizontal
- removed R18, R9: 270, Resistor_THT:R_Axial_DIN0207_L6.3mm_D2.5mm_P10.16mm_Horizontal
- removed R3: 1R 2W, Resistor_THT:R_Axial_DIN0411_L9.9mm_D3.6mm_P12.70mm_Horizontal
- removed R7: 470, Resistor_THT:R_Axial_DIN0207_L6.3mm_D2.5mm_P10.16mm_Horizontal
Routing:
- net SensB: track 42.2 -> 0.00 mm
- net SensA: track 32.7 -> 0.00 mm
- net RelaiBistableSensB_N: track 24.5 -> 0.00 mm
- net RelaiBistableSensA_N: track 19.1 -> 0.00 mm
- net Interrupteur: track 6.10 -> 0.00 mm
- net LED_TractionEnService: track 5.65 -> 0.00 mm
- net LED_Alim: track 5.65 -> 0.00 mm
- net LED_SensB: track 5.44 -> 0.00 mm
- net LED_SensA: track 5.44 -> 0.00 mm
- removed copper zone on F.Cu, net +20V
- removed copper zone on B.Cu, net GND
- removed copper zone on F.Cu, net Traction_P
- removed copper zone on F.Cu, net VCC
Other:
- board outline removed
