File: PCB_IIm_Ligne.kicad_sch (KiCad schematic)
At the start: 42 parts, among them J1 Screw_Terminal_01x08, J2 Screw_Terminal_01x08, J3 Screw_Terminal_01x08, K1 G2RK-2 DC12, K2 Relay_DPDT_Latching_2coil, Q1 MPSA56, Q2 2N2222A, Q3 2N2222A, Q4 2N2222A, Q6 IRF40B207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

Commit message: check BOM
Parts:
- R13, R14: value R10k -> 10K
- R18, R9: value 260 -> 270
- R7: value R1k -> 470
Changed lines of the file:
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@@
 			)
 		)
-		(property "Value" "260"
+		(property "Value" "270"
 			(at 523.24 135.89 90)
 			(show_name no)
@@
 			)
 		)
-		(property "Value" "R1k"
+		(property "Value" "470"
 			(at 113.03 -46.9901 0)
 			(show_name no)
@@
 			)
 		)
-		(property "Value" "260"
+		(property "Value" "270"
 			(at 457.2 135.89 90)
 			(show_name no)
@@
 			)
 		)
-		(property "Value" "R10k"
+		(property "Value" "10K"
 			(at 248.92 -40.6401 0)
 			(show_name no)
@@
 			)
 		)
-		(property "Value" "R10k"
+		(property "Value" "10K"
 			(at 217.17 -16.5101 0)
 			(show_name no)
