File: PCB_IIm_Ligne.kicad_sch (KiCad schematic)
At the start: 43 parts, among them J1 Screw_Terminal_01x08, J2 Screw_Terminal_01x08, J3 Screw_Terminal_01x08, J4 Screw_Terminal_01x08, K2 Relay_DPDT_Latching_2coil, Q1 MPSA56, Q2 2N2222A, Q3 2N2222A, Q4 2N2222A, Q6 IRF40B207, U1 TLC555xP

Commit message: resistance shunt
Connections:
- net +20V: no longer D6.1 (K), R3.1
- net GND: now also R3.2; no longer K1.14 (NO1), K1.22 (NC2)
- net ResistanceShunt: now also D6.1 (K), K1.14 (NO1), K1.22 (NC2), R3.1; no longer R3.2
